Commit message: Motoman has real gripper and it works in gazebo

File: aprs_description/urdf/motoman/aprs_motoman.ros2_control.xacro (robot description, xacro)
@@ -85,4 +85,26 @@
           <state_interface name="effort"/>
       </joint>
+      <joint name="motoman_left_finger_joint">
+          <command_interface name="position">
+            <param name="min">0</param>
+            <param name="max">0.02</param>
+          </command_interface>
+          <state_interface name="position">
+          <param name="initial_value">${initial_positions['left_finger']}</param>
+          </state_interface>
+          <state_interface name="velocity"/>
+          <state_interface name="effort"/>
+      </joint>
+      <joint name="motoman_right_finger_joint">
+          <command_interface name="position">
+          <param name="min">0</param>
+          <param name="max">0.02</param>
+          </command_interface>
+          <state_interface name="position">
+          <param name="initial_value">${initial_positions['right_finger']}</param>
+          </state_interface>
+          <state_interface name="velocity"/>
+          <state_interface name="effort"/>
+      </joint>
     </ros2_control>
   </xacro:macro>

File: aprs_description/urdf/motoman/aprs_motoman_macro.xacro (robot description, xacro)
@@ -9,5 +9,5 @@
     <xacro:include filename="$(find aprs_description)/urdf/motoman/aprs_motoman.ros2_control.xacro"/>
     <!-- Inclue gripper macro -->
-    <xacro:include filename="$(find aprs_description)/urdf/vacuum_gripper/vacuum_gripper_macro.xacro"/>
+    <xacro:include filename="$(find aprs_description)/urdf/motoman/motoman_gripper_macro.xacro"/>
     <xacro:property name="initial_positions_file" default="$(find aprs_description)/config/motoman_initial_positions.yaml"/>
     <!-- Run motoman macro -->
@@ -21,9 +21,5 @@
     </xacro:aprs_motoman_ros2_control>
     <!-- Run gripper macro -->
-    <xacro:vacuum_gripper
-      parent="motoman_gripper_link"
-      prefix="motoman"
-      >
-    </xacro:vacuum_gripper>
+    <xacro:motoman_gripper parent="link_t" />
   </xacro:macro>
 </robot>

File: aprs_description/urdf/motoman/motoman_sia20_macro.xacro (robot description, xacro)
@@ -37,5 +37,4 @@
 			</collision>
 		</link>
-		<link name="motoman_gripper_link"/>
 		<joint name = "motoman_base_joint" type = "fixed">
 			<origin rpy = "0 0 0" xyz = "0 0 0"/>
@@ -201,9 +200,4 @@
 			<xacro:default_joint_misc/>
 		</joint>
-		<joint name = "motoman_link_t_to_gripper" type = "fixed">
-			<origin xyz = "0 0.02 0" rpy = "-1.57 1.57 0"/>
-			<parent link = "link_t"/>
-			<child link = "motoman_gripper_link"/>
-		</joint>
   </xacro:macro>
 </robot>
