Commit message: Picks. Not perfect

File: aprs_description/urdf/aprs_motoman.urdf.xacro (robot description, xacro)
@@ -7,5 +7,5 @@
   <link name="aprs_motoman_base_link"/>
   <joint name = "motoman_world_to_base" type = "fixed">
-    <origin rpy = "0 0 3.14159" xyz = "0.4953 -0.08255 0.9"/>
+    <origin rpy = "0 0 3.14159" xyz = "0.6877125 -0.08255 0.9"/>
     <parent link = "world"/>
     <child link = "aprs_motoman_base_link"/>

File: aprs_description/urdf/fanuc/aprs_fanuc.ros2_control.xacro (robot description, xacro)
@@ -74,4 +74,26 @@
         <state_interface name="effort"/>
       </joint>
+      <joint name="fanuc_left_finger_joint">
+          <command_interface name="position">
+            <param name="min">0</param>
+            <param name="max">0.0075</param>
+          </command_interface>
+          <state_interface name="position">
+          <param name="initial_value">${initial_positions['left_finger']}</param>
+          </state_interface>
+          <state_interface name="velocity"/>
+          <state_interface name="effort"/>
+      </joint>
+      <joint name="fanuc_right_finger_joint">
+          <command_interface name="position">
+          <param name="min">0</param>
+          <param name="max">0.0075</param>
+          </command_interface>
+          <state_interface name="position">
+          <param name="initial_value">${initial_positions['right_finger']}</param>
+          </state_interface>
+          <state_interface name="velocity"/>
+          <state_interface name="effort"/>
+      </joint>
     </ros2_control>
   </xacro:macro>

File: aprs_description/urdf/fanuc/aprs_fanuc_macro.xacro (robot description, xacro)
@@ -9,5 +9,5 @@
     <xacro:include filename="$(find aprs_description)/urdf/fanuc/aprs_fanuc.ros2_control.xacro"/>
     <!-- Inclue gripper macro -->
-    <xacro:include filename="$(find aprs_description)/urdf/vacuum_gripper/vacuum_gripper_macro.xacro"/>
+    <xacro:include filename="$(find aprs_description)/urdf/fanuc/fanuc_gripper_macro.xacro"/>
     <xacro:property name="initial_positions_file" default="$(find aprs_description)/config/fanuc_initial_positions.yaml"/>
     <!-- Run fanuc macro -->
@@ -21,9 +21,5 @@
     </xacro:aprs_fanuc_ros2_control>
     <!-- Run gripper macro -->
-    <xacro:vacuum_gripper
-      parent="fanuc_gripper_link"
-      prefix="fanuc"
-      >
-    </xacro:vacuum_gripper>
+    <xacro:fanuc_gripper parent="link_6" />
   </xacro:macro>
 </robot>

File: aprs_description/urdf/fanuc/fanuc_lrmate200id_macro.xacro (robot description, xacro)
@@ -185,5 +185,4 @@
          </inertial>
       </link>
-      <link name="fanuc_gripper_link"/>
    <!--   <link name="tool0" /> -->
       <joint name = "base_joint_" type = "fixed">
@@ -234,9 +233,4 @@
          <limit effort="${joint6effort}" lower="${joint6lower}" upper="${joint6upper}" velocity="${joint6velocity}" />
       </joint>
-      <joint name = "fanuc_link_6_to_gripper" type = "fixed">
-         <origin xyz = "0 0 0" rpy = "0 1.57 0"/>
-         <parent link = "link_6"/>
-         <child link = "fanuc_gripper_link"/>
-      </joint>
       <gazebo reference="fanuc_base_link">
          <material>Gazebo/Grey</material>
@@ -267,8 +261,4 @@
          <turnGravityOff>true</turnGravityOff>
       </gazebo>
-      <gazebo reference="fanuc_gripper_link">
-         <material>Gazebo/Yellow</material>
-         <turnGravityOff>true</turnGravityOff>
-      </gazebo>
   </xacro:macro>
 </robot>

Commit message: All work done by me

File: aprs_description/urdf/aprs_motoman.urdf.xacro (robot description, xacro)
@@ -7,5 +7,5 @@
   <link name="aprs_motoman_base_link"/>
   <joint name = "motoman_world_to_base" type = "fixed">
-    <origin rpy = "0 0 3.14159" xyz = "0.6877125 -0.08255 0.9"/>
+    <origin rpy = "0 0 3.14159" xyz = "0.6842125 -0.08255 0.9"/>
     <parent link = "world"/>
     <child link = "aprs_motoman_base_link"/>
