Commit message: Updates working with physical robots. Working with motoman. Removed cameras

File: aprs_description/urdf/aprs_fanuc.urdf.xacro (robot description, xacro)
@@ -10,12 +10,6 @@
   <xacro:include filename="$(find aprs_description)/urdf/fanuc/aprs_fanuc_macro.xacro"/>
   <xacro:arg name="fanuc_controller" default="$(find aprs_description)/config/robot_controllers.yaml" />
-  <xacro:arg name="camera_active_arg" default="false"/>
-  <xacro:property name="camera_active" value="$(arg camera_active_arg)" />
-  <xacro:arg name="camera_type_arg" default="rgb"/>
-  <xacro:property name="camera_type" value="$(arg camera_type_arg)" />
   <xacro:aprs_fanuc
     parent="aprs_fanuc_base_link"
-    camera_active="${camera_active}"
-    camera_type="${camera_type}"
     >
   </xacro:aprs_fanuc>

File: aprs_description/urdf/aprs_lab_robots.urdf.xacro (robot description, xacro)
@@ -30,33 +30,15 @@
   <xacro:include filename="$(find aprs_description)/urdf/motoman/aprs_motoman_macro.xacro"/>
   <xacro:arg name="controllers" default="$(find aprs_description)/config/robot_controllers.yaml" />
-  <xacro:arg name="ur_camera_active_arg" default="false"/>
-  <xacro:property name="ur_camera_active" value="$(arg ur_camera_active_arg)" />
-  <xacro:arg name="ur_camera_type_arg" default="rgb"/>
-  <xacro:property name="ur_camera_type" value="$(arg ur_camera_type_arg)" />
   <xacro:aprs_ur
     parent="aprs_ur_base_link"
-    camera_active="${ur_camera_active}"
-    camera_type="${ur_camera_type}"
     >
   </xacro:aprs_ur>
-  <xacro:arg name="fanuc_camera_active_arg" default="false"/>
-  <xacro:property name="fanuc_camera_active" value="$(arg fanuc_camera_active_arg)" />
-  <xacro:arg name="fanuc_camera_type_arg" default="rgb"/>
-  <xacro:property name="fanuc_camera_type" value="$(arg fanuc_camera_type_arg)" />
   <xacro:aprs_fanuc
     parent="aprs_fanuc_base_link"
-    camera_active="${fanuc_camera_active}"
-    camera_type="${fanuc_camera_type}"
     >
   </xacro:aprs_fanuc>
   <xacro:aprs_franka></xacro:aprs_franka>
-  <xacro:arg name="motoman_camera_active_arg" default="false"/>
-  <xacro:property name="motoman_camera_active" value="$(arg motoman_camera_active_arg)" />
-  <xacro:arg name="motoman_camera_type_arg" default="rgb"/>
-  <xacro:property name="motoman_camera_type" value="$(arg motoman_camera_type_arg)" />
   <xacro:aprs_motoman
     parent="aprs_motoman_base_link"
-    camera_active="${motoman_camera_active}"
-    camera_type="${motoman_camera_type}"
     >
   </xacro:aprs_motoman>

File: aprs_description/urdf/aprs_motoman.urdf.xacro (robot description, xacro)
@@ -13,12 +13,6 @@
   <xacro:include filename="$(find aprs_description)/urdf/motoman/aprs_motoman_macro.xacro"/>
   <xacro:arg name="motoman_controller" default="$(find aprs_description)/config/robot_controllers.yaml" />
-  <xacro:arg name="camera_active_arg" default="false"/>
-  <xacro:property name="camera_active" value="$(arg camera_active_arg)" />
-  <xacro:arg name="camera_type_arg" default="rgb"/>
-  <xacro:property name="camera_type" value="$(arg camera_type_arg)" />
   <xacro:aprs_motoman
     parent="aprs_motoman_base_link"
-    camera_active="${camera_active}"
-    camera_type="${camera_type}"
     >
   </xacro:aprs_motoman>

File: aprs_description/urdf/fanuc/aprs_fanuc_macro.xacro (robot description, xacro)
@@ -3,6 +3,4 @@
   <xacro:macro name="aprs_fanuc" params="
     parent
-    camera_active
-    camera_type
 ">
     <!-- Inclue fanuc robot macro -->
@@ -26,6 +24,4 @@
       parent="fanuc_gripper_link"
       prefix="fanuc"
-      use_camera="${camera_active}"
-      camera_type="${camera_type}"
       >
     </xacro:vacuum_gripper>

File: aprs_description/urdf/motoman/aprs_motoman_macro.xacro (robot description, xacro)
@@ -3,6 +3,4 @@
   <xacro:macro name="aprs_motoman" params="
     parent
-    camera_active
-    camera_type
 ">
     <!-- Inclue motoman robot macro -->
@@ -26,6 +24,4 @@
       parent="motoman_gripper_link"
       prefix="motoman"
-      use_camera="${camera_active}"
-      camera_type="${camera_type}"
       >
     </xacro:vacuum_gripper>

File: aprs_description/urdf/ur/aprs_ur_macro.xacro (robot description, xacro)
@@ -34,12 +34,4 @@
       </plugin>
     </gazebo>
-    <!-- Run gripper macro -->
-    <!-- <xacro:vacuum_gripper
-      parent="tool0"
-      prefix="ur"
-      use_camera="${camera_active}"
-      camera_type="${camera_type}"
-      >
-    </xacro:vacuum_gripper> -->
   </xacro:macro>
 </robot>

File: aprs_description/urdf/vacuum_gripper/vacuum_gripper_macro.xacro (robot description, xacro)
@@ -4,6 +4,4 @@
     parent
     prefix
-    use_camera
-    camera_type
     ">
     <!-- Gripper Link -->
@@ -50,127 +48,4 @@
       </sensor>
     </gazebo>
-    <!-- Camera -->
-    <xacro:if value="${use_camera}">
-      <!-- Mount Link -->
-      <link name ="${prefix}_robot_camera_mount_link">
-        <visual>
-          <origin xyz="0 0 0" rpy="0 0 0"/>
-          <geometry>
-            <mesh filename="file://$(find aprs_description)/meshes/vacuum_gripper/camera_mount.stl" scale="1 1 1"/>
-          </geometry>
-        </visual>
-      </link>
-      <!-- Camera Link -->
-      <link name ="${prefix}_robot_camera_link">
-        <visual>
-          <origin xyz="0 0 0" rpy="1.57 0 1.57"/>
-          <geometry>
-            <mesh filename="file://$(find aprs_description)/meshes/vacuum_gripper/camera.stl" scale="1 1 1"/>
-          </geometry>
-        </visual>
-      </link>
-      <link name ="${prefix}_robot_camera_optical_link">
-      </link>
-      <!-- Add camera mount joint -->
-      <joint name="${prefix}_robot_camera_mount_joint" type="fixed">
-        <axis xyz="0 1 0" />
-        <origin xyz="0 0 -0.012" rpy="0 0 0"/>
-        <parent link="${prefix}_gripper"/>
-        <child link="${prefix}_robot_camera_mount_link"/>
-      </joint>
-      <!-- Add camera joint -->
-      <joint name="${prefix}_robot_camera_joint" type="fixed">
-        <axis xyz="0 1 0" />
-        <origin xyz="0 -.07 -.006" rpy="0 -1.57 1.57"/>
-        <parent link="${prefix}_robot_camera_mount_link"/>
-        <child link="${prefix}_robot_camera_link"/>
-      </joint>
-      <!-- Add optical joint -->
-      <joint name="${prefix}_robot_camera_optical_joint" type="fixed">
-        <axis xyz="0 1 0" />
-        <origin xyz="0 0 0" rpy="-1.57 0 -1.57"/>
-        <parent link="${prefix}_robot_camera_link"/>
-        <child link="${prefix}_robot_camera_optical_link"/>
-      </joint>
-      <!-- Add color to links -->
-      <gazebo reference="${prefix}_robot_camera_mount_link">
-        <material>Gazebo/Black</material>
-      </gazebo>
-      <gazebo reference="${prefix}_robot_camera_link">
-        <material>Gazebo/White</material>
-      </gazebo>
-      <!-- Add gazebo sensors -->
-      <xacro:property name="type" value="${camera_type}"/>
-      <gazebo reference="${prefix}_robot_camera_link">
-        <!-- Add rgb camera -->
-        <xacro:if value="${type == 'rgb'}">
-          <sensor type="camera" name="rgb_camera">
-            <topic>${prefix}_robot_rgb_camera_gz_topic</topic>
-            <always_on>true</always_on>
-            <visualize>false</visualize>
-            <update_rate>15</update_rate>
-            <camera name="${prefix}_robot_camera">
-              <horizontal_fov>1.5</horizontal_fov>
-              <image>
-                <width>640</width>
-                <height>480</height>
-                <format>R8G8B8</format>
-              </image>
-              <clip>
-                <near>0.1</near>
-                <far>10</far>
-              </clip>
-            </camera>
-            <plugin name="ariac_sensors::AriacCameraPlugin" filename="libAriacCameraPlugin.so">
-              <ros>
-                <namespace></namespace>
-              </ros>
-              <camera_type>rgb</camera_type>
-              <gz_topic>${prefix}_robot_rgb_camera_gz_topic</gz_topic>
-              <camera_name>${prefix}_robot_rgb_camera</camera_name>
-              <rgb_img_ros_topic>/ariac/sensors/${prefix}_robot_rgb_camera/rgb_image</rgb_img_ros_topic>
-              <cam_info_ros_topic>/ariac/sensors/${prefix}_robot_rgb_camera/camera_info</cam_info_ros_topic>
-              <cam_info_gz_topic>${prefix}_robot_rgb_camera_gz_topic_info</cam_info_gz_topic>
-            </plugin>
-          </sensor>
-        </xacro:if>
-        <xacro:if value="${type == 'rgbd'}">
-          <sensor type="depth" name="rgbd_camera">
-            <topic>${prefix}_robot_rgbd_camera_gz_topic</topic>
-            <always_on>true</always_on>
-            <visualize>false</visualize>
-            <update_rate>15</update_rate>
-            <camera name="${prefix}_robot_camera">
-              <horizontal_fov>1.5</horizontal_fov>
-              <image>
-                <width>640</width>
-                <height>480</height>
-                <format>R8G8B8</format>
-              </image>
-              <clip>
-                <near>0.1</near>
-                <far>10</far>
-              </clip>
-              <noise>
-                <type>gaussian</type>
-                <mean>0.0</mean>
-                <stddev>0.001</stddev>
-              </noise>
-            </camera>
-            <plugin name="ariac_sensors::AriacCameraPlugin" filename="libAriacCameraPlugin.so">
-              <ros>
-                <namespace></namespace>
-              </ros>
-              <camera_type>rgbd</camera_type>
-              <camera_name>${prefix}_robot_rgbd_camera</camera_name>
-              <gz_topic>${prefix}_robot_rgbd_camera_gz_topic</gz_topic>
-              <rgb_img_ros_topic>/ariac/sensors/${prefix}_robot_rgbd_camera/rgb_image</rgb_img_ros_topic>
-              <depth_img_ros_topic>/ariac/sensors/${prefix}_robot_rgbd_camera/depth_image</depth_img_ros_topic>
-              <cam_info_ros_topic>/ariac/sensors/${prefix}_robot_rgbd_camera/camera_info</cam_info_ros_topic>
-            </plugin>
-          </sensor>
-        </xacro:if>
-      </gazebo>
-    </xacro:if>
   </xacro:macro>
 </robot>

Commit message: Real time up to 86

File: aprs_description/urdf/aprs_fanuc.urdf.xacro (robot description, xacro)
@@ -4,5 +4,5 @@
   <link name="aprs_fanuc_base_link"/>
   <joint name = "fanuc_world_to_base" type = "fixed">
-    <origin rpy = "0 0 0" xyz = "-0.5222875 -0.073025 0.84455"/>
+    <origin rpy = "0 0 0" xyz = "-0.5222875 -0.073025 0.88"/>
     <parent link = "world"/>
     <child link = "aprs_fanuc_base_link"/>

File: aprs_description/urdf/aprs_franka.urdf.xacro (robot description, xacro)
@@ -3,5 +3,5 @@
   <link name="world"/>
   <joint name = "franka_world_to_base" type = "fixed">
-    <origin rpy = "0 0 0" xyz = "-1.3145625 -1.375 0.8397875"/>
+    <origin rpy = "0 0 0" xyz = "-1.3145625 -1.375 0.85"/>
     <parent link = "world"/>
     <child link = "aprs_franka_base_link"/>

Commit message: Trays and gears spawn in automatically when mirror_env is true. Grippers now don'd depend on other repositories. Recentered environment

File: aprs_description/urdf/aprs_fanuc.urdf.xacro (robot description, xacro)
@@ -4,5 +4,5 @@
   <link name="aprs_fanuc_base_link"/>
   <joint name = "fanuc_world_to_base" type = "fixed">
-    <origin rpy = "0 0 0" xyz = "-0.5222875 -0.073025 0.88"/>
+    <origin rpy = "0 0 0" xyz = "0.756925 0.1759 -0.03045"/>
     <parent link = "world"/>
     <child link = "aprs_fanuc_base_link"/>

File: aprs_description/urdf/aprs_franka.urdf.xacro (robot description, xacro)
@@ -3,5 +3,5 @@
   <link name="world"/>
   <joint name = "franka_world_to_base" type = "fixed">
-    <origin rpy = "0 0 0" xyz = "-1.3145625 -1.375 0.85"/>
+    <origin rpy = "0 0 0" xyz = "-0.03535 -1.126075 -0.0352125"/>
     <parent link = "world"/>
     <child link = "aprs_franka_base_link"/>

File: aprs_description/urdf/aprs_lab_robots.urdf.xacro (robot description, xacro)
@@ -6,20 +6,20 @@
   <link name="aprs_motoman_base_link"/>
   <joint name = "ur_world_to_base" type = "fixed">
-    <origin rpy = "0 0 0" xyz = "0.7864625 -1.375 0.8001"/>
+    <origin rpy = "0 0 0" xyz = "2.065675 -1.126075 -0.0749"/>
     <parent link = "world"/>
     <child link = "aprs_ur_base_link"/>
   </joint>
   <joint name = "fanuc_world_to_base" type = "fixed">
-    <origin rpy = "0 0 0" xyz = "-0.5222875 -0.073025 0.84455"/>
+    <origin rpy = "0 0 0" xyz = "0.756925 0.1759 -0.03045"/>
     <parent link = "world"/>
     <child link = "aprs_fanuc_base_link"/>
   </joint>
   <joint name = "franka_world_to_base" type = "fixed">
-    <origin rpy = "0 0 0" xyz = "-1.3145625 -1.375 0.8397875"/>
+    <origin rpy = "0 0 0" xyz = "-0.03535 -1.126075 -0.0352125"/>
     <parent link = "world"/>
     <child link = "aprs_franka_base_link"/>
   </joint>
   <joint name = "motoman_world_to_base" type = "fixed">
-    <origin rpy = "0 0 3.14159" xyz = "0.4953 -0.08255 0.9"/>
+    <origin rpy = "0 0 3.14159" xyz = "1.7745125 0.166375 0.025"/>
     <parent link = "world"/>
     <child link = "aprs_motoman_base_link"/>

File: aprs_description/urdf/aprs_motoman.urdf.xacro (robot description, xacro)
@@ -7,5 +7,5 @@
   <link name="aprs_motoman_base_link"/>
   <joint name = "motoman_world_to_base" type = "fixed">
-    <origin rpy = "0 0 3.14159" xyz = "0.6842125 -0.08255 0.9"/>
+    <origin rpy = "0 0 3.14159" xyz = "1.963425 0.166375 0.025"/>
     <parent link = "world"/>
     <child link = "aprs_motoman_base_link"/>

File: aprs_description/urdf/aprs_ur.urdf.xacro (robot description, xacro)
@@ -4,5 +4,5 @@
   <link name="aprs_ur_base_link"/>
   <joint name = "ur_world_to_base" type = "fixed">
-    <origin rpy = "0 0 0" xyz = "0.7864625 -1.375 0.8001"/>
+    <origin rpy = "0 0 0" xyz = "2.065675 -1.126075 -0.0749"/>
     <parent link = "world"/>
     <child link = "aprs_ur_base_link"/>

File: aprs_description/urdf/fanuc/fanuc_gripper_macro.xacro (robot description, xacro)
@@ -9,5 +9,5 @@
         <origin rpy="0 0 0" xyz="0 0 0" />
         <geometry>
-          <mesh filename="file://$(find fanuc_description)/meshes/gripper_link.stl"/>
+          <mesh filename="file://$(find aprs_description)/meshes/fanuc/gripper/gripper_link.stl"/>
         </geometry>
         <material name="">
@@ -18,5 +18,5 @@
         <origin rpy="0 0 0" xyz="0 0 0" />
         <geometry>
-          <mesh filename="file://$(find fanuc_description)/meshes/gripper_link.stl" />
+          <mesh filename="file://$(find aprs_description)/meshes/fanuc/gripper/gripper_link.stl" />
         </geometry>
       </collision>
@@ -32,5 +32,5 @@
         <origin xyz="0 0 0" rpy="0 0 0" />
         <geometry>
-          <mesh filename="file://$(find fanuc_description)/meshes/fanuc_left_finger.stl" />
+          <mesh filename="file://$(find aprs_description)/meshes/fanuc/gripper/fanuc_left_finger.stl" />
         </geometry>
         <material name="">
@@ -41,5 +41,5 @@
         <origin rpy="0 0 0" xyz="0 0 0" />
         <geometry>
-          <mesh filename="file://$(find fanuc_description)/meshes/fanuc_left_finger.stl" />
+          <mesh filename="file://$(find aprs_description)/meshes/fanuc/gripper/fanuc_left_finger.stl" />
         </geometry>
       </collision>
@@ -55,5 +55,5 @@
         <origin xyz="0 0 0" rpy="0 0 0" />
         <geometry>
-          <mesh filename="file://$(find fanuc_description)/meshes/fanuc_right_finger.stl" />
+          <mesh filename="file://$(find aprs_description)/meshes/fanuc/gripper/fanuc_right_finger.stl" />
         </geometry>
         <material name="">
@@ -64,5 +64,5 @@
         <origin rpy="0 0 0" xyz="0 0 0" />
         <geometry>
-          <mesh filename="file://$(find fanuc_description)/meshes/fanuc_right_finger.stl" />
+          <mesh filename="file://$(find aprs_description)/meshes/fanuc/gripper/fanuc_right_finger.stl" />
         </geometry>
       </collision>

File: aprs_description/urdf/motoman/motoman_gripper_macro.xacro (robot description, xacro)
@@ -9,5 +9,5 @@
         <origin rpy="0 0 0" xyz="0 0 0" />
         <geometry>
-          <mesh filename="file://$(find motoman_description)/meshes/motoman_gripper_link_simplified.stl"/>
+          <mesh filename="file://$(find aprs_description)/meshes/motoman/gripper/motoman_gripper_link_simplified.stl"/>
         </geometry>
         <material name="">
@@ -18,5 +18,5 @@
         <origin rpy="0 0 0" xyz="0 0 0" />
         <geometry>
-          <mesh filename="file://$(find motoman_description)/meshes/motoman_gripper_link_simplified.stl" />
+          <mesh filename="file://$(find aprs_description)/meshes/motoman/gripper/motoman_gripper_link_simplified.stl" />
         </geometry>
       </collision>
@@ -32,8 +32,8 @@
         <origin xyz="0 0 0" rpy="0 0 0" />
         <geometry>
-          <mesh filename="file://$(find motoman_description)/meshes/motoman_left_finger.stl" />
+          <mesh filename="file://$(find aprs_description)/meshes/motoman/gripper/motoman_left_finger.stl" />
         </geometry>
         <material name="">
-          <color rgba="0.79216 0.81961 0.93333 1" />
+          <color rgba="0.79216 0.81961 0.93333 1"/>
         </material>
       </visual>
@@ -41,5 +41,5 @@
         <origin rpy="0 0 0" xyz="0 0 0" />
         <geometry>
-          <mesh filename="file://$(find motoman_description)/meshes/motoman_left_finger.stl" />
+          <mesh filename="file://$(find aprs_description)/meshes/motoman/gripper/motoman_left_finger.stl" />
         </geometry>
       </collision>
@@ -55,5 +55,5 @@
         <origin xyz="0 0 0" rpy="0 0 0" />
         <geometry>
-          <mesh filename="file://$(find motoman_description)/meshes/motoman_right_finger.stl" />
+          <mesh filename="file://$(find aprs_description)/meshes/motoman/gripper/motoman_right_finger.stl" />
         </geometry>
         <material name="">
@@ -64,5 +64,5 @@
         <origin rpy="0 0 0" xyz="0 0 0" />
         <geometry>
-          <mesh filename="file://$(find motoman_description)/meshes/motoman_right_finger.stl" />
+          <mesh filename="file://$(find aprs_description)/meshes/motoman/gripper/motoman_right_finger.stl" />
         </geometry>
       </collision>
